File: Zx50_MemoryCard_RevA.kicad_pcb (KiCad board)
At the start: 4 copper layers, 123.1 x 129.8 mm, 53 parts, among them J1 Zx50_EdgeConnector, J2 JTAG, SW1 SW_DIP_x05, U1 SN74ABT541BN, U10 CY7C1049GN, U11 CY7C1049GN, U12 SST39SF040, U2 74AHCT1G04, U3 SN74ABT16244ADL, U4 74ABT245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

Commit message: RevA.6 as sent to fab.
Parts:
- moved C8 65.8 mm to (44.2, 36.6), turned to 90 degrees
- moved C3 51.0 mm to (90.2, 125.8), turned to -90 degrees
- moved C9 48.9 mm to (54.5, 89.5), turned to 0 degrees
- moved C27 7.24 mm to (69.2, 59.1)
- moved C26 6.91 mm to (69.2, 52.1)
- moved U1 2.40 mm to (94.7, 127.7)
- moved C23 1.98 mm to (115.1, 108.7)
- moved C5 0.18 mm to (64.6, 94.9)
- moved C6 0.13 mm to (68.2, 106.7)
- moved C7 0.10 mm to (68.4, 125.7)
- moved C4 0.08 mm to (68.3, 74.3)
- renumbered C14 to C13, C13 to C14
Connections:
- C3 pad 1: (no net) -> +5V
- C3 pad 2: (no net) -> GND
- C4 pad 1: (no net) -> +5V
- C4 pad 2: (no net) -> GND
- C5 pad 1: (no net) -> +5V
- C5 pad 2: (no net) -> GND
Routing:
- net /B.D3: track 208.4 -> 284.1 mm, vias 5 -> 7
- net /B.D2: track 222.1 -> 297.9 mm, vias 5 -> 7
- net /B.D1: track 215.9 -> 291.0 mm, vias 5 -> 7
- net /B.D0: track 213.1 -> 287.4 mm, vias 5 -> 7
- net /B.D4: track 203.5 -> 277.4 mm, vias 5 -> 7
- net /B.D5: track 203.3 -> 275.2 mm, vias 5 -> 7
- net /B.D6: track 196.7 -> 266.7 mm, vias 5 -> 7
- net /B.D7: track 196.3 -> 265.0 mm, vias 5 -> 7
- net /~SH_D_OE~: track 59.9 -> 69.3 mm, vias 0 -> 2
- net /~SH_BUSY~: track 79.6 -> 88.5 mm, vias 1 -> 3
- net /B.SH_RW: track 48.6 -> 56.7 mm, vias 0 -> 2
- net /B.~SH_DONE~: track 50.2 -> 58.0 mm, vias 0 -> 2
- net /B.~SH_EN~: track 47.2 -> 53.9 mm, vias 0 -> 2
- net /B.~SH_INC~: track 45.9 -> 52.0 mm, vias 0 -> 2
- net /SH_C_DIR: track 52.1 -> 57.9 mm, vias 0 -> 2
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- added copper zone on F.Cu, net +5V
Other:
- board size 123.1 x 129.8 mm -> 123.4 x 129.8 mm
- board text added: "Zx50 RAM/ROM with DMA Burst Dual Phase Shadow Bus Marc Mosko, 2026 Zx50_MemoryCard_RevA.6"
- board text removed: "Zx50 RAM/ROM with DMA Burst Dual Phase Shadow Bus Marc Mosko, 2026 Zx50_MemoryCard_RevA"
