File: Zx50_MemoryCard_RevA/Zx50_MemoryCard_RevA.kicad_sch (KiCad schematic)
At the start: 21 parts, among them J1 Zx50_EdgeConnector, SW1 SW_DIP_x05, U1 SN74ABT541BN, U2 74AHCT1G04, U3 SN74ABT16244ADL, U4 74ABT245, U5 SN74ABT541BN, U6 74ABT245, U7 74ABT245

Commit message: move files in big reorg
Parts:
- C1, C2, C26, C27, C3, C4, C5, C6, C7, C8, C9, U1, U2, U3, U4, U5, U6, U7: now left out of the parts list
- J1: DigiKey_PN (none) -> 2057-PH2RA-80-UA-ND; SKU (none) -> PH2RA-80-UA
- RN1: DigiKey_PN (none) -> 4606X-AP1-103LFCT-ND; LCSC (none) -> 4606X-AP1-103LF
- SW1: DigiKey_PN (none) -> CT2085-ND; LCSC (none) -> 208-5
