File: Zx50_MemoryCard_RevA/cpld_mem_RevA.kicad_sch (KiCad schematic)
At the start: 32 parts, among them J2 JTAG, U10 CY7C1049GN, U11 CY7C1049GN, U12 SST39SF040, U8 ATF1508AS-10AU100, U9 IS61C256AL-12JLI

Commit message: move files in big reorg
Parts:
- added MISC1: ~, DIP-32 socket, symbol zx50_symbols:DIP-32_Socket
- C10, C11, C12, C13, C14, C15, C16, C17, C18, C19, C20, C21, C22, C23, C24, C25, D1, D2, D3, D4, D5, R1, R2, R3, R4, R5, U10, U11, U8, U9: now left out of the parts list
- J2: DigiKey_PN (none) -> 732-2094-ND; SKU (none) -> 61201021621
- U12: DigiKey_PN (none) -> SST39SF040-70-4C-PHE-ND; SKU (none) -> SST39SF040-70-4C-PHE
