File: Zx50_Cpu/Zx50_Cpu.kicad_sch (KiCad schematic)
At the start: 23 parts, among them J1 Zx50_EdgeConnector, J2 FrontPanelConnect, J3 Clock Mezzanine, J4 Front Panel, SW1 RESET, U1 74AHC1G14, U2 SN74AHCT245N, U3 SN74AHCT245N, U4 Z84C00xxP, U5 SN74AHCT245N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

Commit message: before routing
Parts:
- added C9: 10uF, Capacitor_THT:CP_Radial_Tantal_D5.0mm_P2.50mm, symbol zx50_symbols:C_10uF_Tant
Connections:
- net +5V: now also C9.1
- net A0: now also U2.9 (A8); no longer U2.2 (A1)
- net A1: now also U2.8 (A7); no longer U2.3 (A2)
- net A10: now also U3.7 (A6); no longer U3.4 (A3)
- net A11: now also U3.6 (A5); no longer U3.5 (A4)
- net A12: now also U3.5 (A4); no longer U3.6 (A5)
- net A13: now also U3.4 (A3); no longer U3.7 (A6)
- net A14: now also U3.3 (A2); no longer U3.8 (A7)
- net A15: now also U3.2 (A1); no longer U3.9 (A8)
- net A2: now also U2.7 (A6); no longer U2.4 (A3)
- net A3: now also U2.6 (A5); no longer U2.5 (A4)
- net A4: now also U2.5 (A4); no longer U2.6 (A5)
- net A5: now also U2.4 (A3); no longer U2.7 (A6)
- net A6: now also U2.3 (A2); no longer U2.8 (A7)
- net A7: now also U2.2 (A1); no longer U2.9 (A8)
- net A8: now also U3.9 (A8); no longer U3.2 (A1)
- net A9: now also U3.8 (A7); no longer U3.3 (A2)
- net BUS.A0: now also U2.11 (B8); no longer U2.18 (B1)
- net BUS.A1: now also U2.12 (B7); no longer U2.17 (B2)
- net BUS.A10: now also U3.13 (B6); no longer U3.16 (B3)
- net BUS.A11: now also U3.14 (B5); no longer U3.15 (B4)
- net BUS.A12: now also U3.15 (B4); no longer U3.14 (B5)
- net BUS.A13: now also U3.16 (B3); no longer U3.13 (B6)
- net BUS.A14: now also U3.17 (B2); no longer U3.12 (B7)
- net BUS.A15: now also U3.18 (B1); no longer U3.11 (B8)
- net BUS.A2: now also U2.13 (B6); no longer U2.16 (B3)
- net BUS.A3: now also U2.14 (B5); no longer U2.15 (B4)
- net BUS.A4: now also U2.15 (B4); no longer U2.14 (B5)
- net BUS.A5: now also U2.16 (B3); no longer U2.13 (B6)
- net BUS.A6: now also U2.17 (B2); no longer U2.12 (B7)
- net BUS.A7: now also U2.18 (B1); no longer U2.11 (B8)
- net BUS.A8: now also U3.11 (B8); no longer U3.18 (B1)
- net BUS.A9: now also U3.12 (B7); no longer U3.17 (B2)
- net BUS.D0: now also U5.11 (B8); no longer U5.18 (B1)
- net BUS.D1: now also U5.12 (B7); no longer U5.17 (B2)
- net BUS.D2: now also U5.13 (B6); no longer U5.16 (B3)
- net BUS.D3: now also U5.14 (B5); no longer U5.15 (B4)
- net BUS.D4: now also U5.15 (B4); no longer U5.14 (B5)
- net BUS.D5: now also U5.16 (B3); no longer U5.13 (B6)
- net BUS.D6: now also U5.17 (B2); no longer U5.12 (B7)
- net BUS.D7: now also U5.18 (B1); no longer U5.11 (B8)
- net BUS.~HALT~: now also U7.18 (B1); no longer U7.12 (B7)
- net BUS.~M1~: now also U7.16 (B3); no longer U7.14 (B5)
- net BUS.~MREQ~: now also U7.14 (B5); no longer U7.16 (B3)
- net BUS.~RD~: now also U7.12 (B7); no longer U7.18 (B1)
- net BUS.~RFSH~: now also U7.17 (B2); no longer U7.13 (B6)
- net BUS.~WR~: now also U7.13 (B6); no longer U7.17 (B2)
- net D0: now also U5.9 (A8); no longer U5.2 (A1)
- net D1: now also U5.8 (A7); no longer U5.3 (A2)
- net D2: now also U5.7 (A6); no longer U5.4 (A3)
- net D3: now also U5.6 (A5); no longer U5.5 (A4)
- net D4: now also U5.5 (A4); no longer U5.6 (A5)
- net D5: now also U5.4 (A3); no longer U5.7 (A6)
- net D6: now also U5.3 (A2); no longer U5.8 (A7)
- net D7: now also U5.2 (A1); no longer U5.9 (A8)
- net GND: now also C9.2
- net ~HALT~: now also U7.2 (A1); no longer U7.8 (A7)
- net ~M1~: now also U7.4 (A3); no longer U7.6 (A5)
- net ~MREQ~: now also U7.6 (A5); no longer U7.4 (A3)
- net ~RD~: now also U7.8 (A7); no longer U7.2 (A1)
- net ~RFSH~: now also U7.3 (A2); no longer U7.7 (A6)
- net ~WR~: now also U7.7 (A6); no longer U7.3 (A2)
