File: Zx50_Cpu/Zx50_Cpu.kicad_sch (KiCad schematic)
At the start: 24 parts, among them J1 Zx50_EdgeConnector, J2 FrontPanelConnect, J3 Clock Mezzanine, J4 Front Panel, SW1 RESET, U1 74AHC1G14, U2 SN74AHCT245N, U3 SN74AHCT245N, U4 Z84C00xxP, U5 SN74AHCT245N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

Commit message: add mounting holes
Parts:
- J1: footprint zx50_footprints:PinHeader_2x40_P2.54mm_Horizontal_Edge -> Connector_PinSocket_2.54mm:PinSocket_2x40_P2.54mm_Vertical_Oval; DigiKey_PN (none) -> A34273-40-ND
- J2: DigiKey_PN (none) -> S1012E-02-ND
- J3, J4: symbol Connector_Generic:Conn_02x05_Odd_Even -> zx50_symbols:Conn_02x05_Odd_Even; DigiKey_PN (none) -> 732-2098-ND
- U2, U3, U5: DigiKey_PN (none) -> 296-1476-5-ND
- U6: footprint Package_TO_SOT_SMD:SOT-23-5_HandSoldering -> SOT-23-5_MC_MCH; DigiKey_PN (none) -> MCP1318MT-46LE/OTCT-ND; Digikey_PN MCP1318MT-46LE/OTCT-ND -> (none)
- U7: DigiKey_PN (none) -> 296-1476-5-ND; Digikey_PN 296-1476-5-ND -> (none)
Changed lines of the file:
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@@
 			)
 		)
+		(property "DigiKey_PN" "296-1476-5-ND"
+			(at 44.45 111.76 90)
+			(effects
+				(font
+					(size 1.27 1.27)
+				)
+				(hide yes)
+			)
+		)
 		(pin "8"
 		)
@@
 			)
 		)
-		(property "Datasheet" ""
+		(property "Datasheet" "~"
 			(at 222.25 96.52 0)
 			(effects
@@
 			)
 		)
-		(property "Description" ""
+		(property "Description" "Resistor, small symbol"
 			(at 222.25 96.52 0)
 			(effects
@@
 			)
 		)
-		(property "Footprint" "Package_TO_SOT_SMD:SOT-23-5_HandSoldering"
+		(property "Footprint" "SOT-23-5_MC_MCH"
 			(at 194.31 60.96 0)
 			(effects
@@
 			)
 		)
-		(property "Digikey_PN" "MCP1318MT-46LE/OTCT-ND"
+		(property "DigiKey_PN" "MCP1318MT-46LE/OTCT-ND"
 			(at 194.31 60.96 0)
 			(effects
@@
 			)
 		)
-		(property "Footprint" "zx50_footprints:PinHeader_2x40_P2.54mm_Horizontal_Edge"
+		(property "Footprint" "Connector_PinSocket_2.54mm:PinSocket_2x40_P2.54mm_Vertical_Oval"
 			(at 128.524 170.18 0)
 			(effects
@@
 			)
 		)
-		(property "Datasheet" ""
+		(property "Datasheet" "~"
 			(at 73.66 180.34 0)
 			(effects
@@
 			)
 		)
-		(property "Description" ""
+		(property "Description" "Generic connector, double row, 02x40, odd/even pin numbering scheme (row 1 odd numbers, row 2 even numbers), script generated (kicad-library-utils/schlib/autogen/connector/)"
 			(at 131.572 173.736 0)
 			(effects
@@
 			)
 		)
+		(property "DigiKey_PN" "A34273-40-ND"
+			(at 73.66 180.34 0)
+			(effects
+				(font
+					(size 1.27 1.27)
+				)
+				(hide yes)
+			)
+		)
 		(pin "41"
 		)
@@
 	)
 	(symbol
-		(lib_id "Connector_Generic:Conn_02x05_Odd_Even")
+		(lib_id "zx50_symbols:Conn_02x05_Odd_Even")
 		(at 256.54 85.09 0)
 		(unit 1)
@@
 			)
 		)
+		(property "DigiKey_PN" "732-2098-ND"
+			(at 256.54 85.09 0)
+			(effects
+				(font
+					(size 1.27 1.27)
+				)
+				(hide yes)
+			)
+		)
 		(pin "3"
 		)
@@
 			)
 		)
+		(property "DigiKey_PN" "S1012E-02-ND"
+			(at 124.46 152.4 90)
+			(effects
+				(font
+					(size 1.27 1.27)
+				)
+				(hide yes)
+			)
+		)
 		(pin "1"
 		)
@@
 	)
 	(symbol
-		(lib_id "Connector_Generic:Conn_02x05_Odd_Even")
+		(lib_id "zx50_symbols:Conn_02x05_Odd_Even")
 		(at 256.54 63.5 0)
 		(unit 1)
@@
 			)
 		)
+		(property "DigiKey_PN" "732-2098-ND"
+			(at 256.54 63.5 0)
+			(effects
+				(font
+					(size 1.27 1.27)
+				)
+				(hide yes)
+			)
+		)
 		(pin "5"
 		)
@@
 			)
 		)
+		(property "DigiKey_PN" "296-1476-5-ND"
+			(at 157.48 111.76 90)
+			(effects
+				(font
+					(size 1.27 1.27)
+				)
+				(hide yes)
+			)
+		)
 		(pin "8"
 		)
@@
 			)
 		)
+		(property "DigiKey_PN" "296-1476-5-ND"
+			(at 102.87 111.76 90)
+			(effects
+				(font
+					(size 1.27 1.27)
+				)
+				(hide yes)
+			)
+		)
 		(pin "8"
 		)
@@
 			)
 		)
-		(property "Digikey_PN" "296-1476-5-ND"
-			(at 219.71 116.84 0)
+		(property "DigiKey_PN" "296-1476-5-ND"
+			(at 219.71 111.76 90)
 			(effects
 				(font

Commit message: finish up cpu card, begin on serial card.
Parts:
- J3: DigiKey_PN 732-2098-ND -> S5558-ND; SKU (none) -> PPPC052LJBN-RC
Changed lines of the file:
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@@
 			)
 		)
-		(property "DigiKey_PN" "732-2098-ND"
+		(property "DigiKey_PN" "S5558-ND"
 			(at 256.54 63.5 0)
 			(effects
+				(font
+					(size 1.27 1.27)
+				)
+				(hide yes)
+			)
+		)
+		(property "SKU" "	 PPPC052LJBN-RC"
+			(at 256.54 63.5 0)
+			(effects
